File: pcb/moisture-sensor.kicad_pcb (KiCad board)
At the start: 2 copper layers, 40 x 125 mm, 35 parts, among them J3 USB4110, U1 ESP32-C3-WROOM-02, U2 TPS631000, U4 MCP73832, Y1 32.768kHz

Commit message: improve PCB
Parts:
- RESET1: footprint library:Panasonic_Electronic_Components-EVQ-P2202M-MFG -> Button_Switch_SMD:SW_SPST_EVQP2
- U2: footprint friedrich:SOT-583 -> Package_TO_SOT_SMD:SC-70-8
- moved J3 0.64 mm to (148.0, 74.0)
- turned R6 to 180 degrees
- turned RESET1 to 90 degrees
- turned U2 to 0 degrees
Connections:
- RESET1 pad 1: Net-(R4-Pad1) -> GND
- RESET1 pad 2: GND -> Net-(R4-Pad1)
Routing:
- net Net-(R4-Pad1): track 25.5 -> 23.9 mm
- net /USB_D-: track 31.8 -> 33.4 mm, vias 0 -> 2
- net +3.3V: track 76.2 -> 75.1 mm
- net Net-(J3-PadB5): track 12.1 -> 13.2 mm
- net Net-(J3-PadA5): track 8.91 -> 9.69 mm
- net /USB_D+: track 35.7 -> 36.0 mm, vias 2 -> 0
- net GND: vias 73 -> 74

Commit message: add footprints and 3d models, increase solder pad size
Parts:
- U1: footprint Espressif:ESP32-C3-WROOM-02 -> library:ESP32-C3-WROOM-02
- Y1: footprint library:XTAL_ABS07-32.768KHZ-1-T -> library:ABS07-32.768KHZ-T
Routing:
- net /USB_D+: track 36.0 -> 36.6 mm
- net GND: vias 74 -> 73

Commit message: adjust some component values
Parts:
- C4: value 22uF -> 47uF
- R12: value 120R -> 220R
Changed lines of the file:
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@@
     (descr "Resistor SMD 0805 (2012 Metric), square (rectangular) end terminal, IPC_7351 nominal with elongated pad for handsoldering. (Body size source: IPC-SM-782 page 72, https://www.pcb-3d.com/wordpress/wp-content/uploads/ipc-sm-782a_amendment_1_and_2.pdf), generated with kicad-footprint-generator")
     (tags "resistor handsolder")
-    (property "MPN" "RC0805FR-07120RL")
+    (property "MPN" "RC0805FR-07220RL")
     (property "Sheetfile" "File: moisture-sensor.kicad_sch")
     (property "Sheetname" "")
@@
       (effects (font (size 1 1) (thickness 0.15)))
     )
-    (fp_text value "120R" (at 0 1.65) (layer "F.Fab")
+    (fp_text value "220R" (at 0 1.65) (layer "F.Fab")
       (effects (font (size 1 1) (thickness 0.15)))
     )
@@
     (descr "Capacitor SMD 0805 (2012 Metric), square (rectangular) end terminal, IPC_7351 nominal with elongated pad for handsoldering. (Body size source: IPC-SM-782 page 76, https://www.pcb-3d.com/wordpress/wp-content/uploads/ipc-sm-782a_amendment_1_and_2.pdf, https://docs.google.com/spreadsheets/d/1BsfQQcO9C6DZCsRaXUlFlo91Tg2WpOkGARC1WS5S8t0/edit?usp=sharing), generated with kicad-footprint-generator")
     (tags "capacitor handsolder")
-    (property "MPN" "GRM21BZ71A226ME15")
+    (property "MPN" "GRM21BR61A476ME15")
     (property "Sheetfile" "File: moisture-sensor.kicad_sch")
     (property "Sheetname" "")
@@
       (effects (font (size 1 1) (thickness 0.15)))
     )
-    (fp_text value "22uF" (at 0 1.68) (layer "F.Fab")
-      (effects (font (size 1 1) (thickness 0.15)))
-    )
+    (fp_text value "47uF" (at 0 1.68) (layer "F.Fab")
+      (effects (font (size 1 1) (thickness 0.15)))
+    )

Commit message: add battery text
Other:
- board text added: "Battery"
Changed lines of the file:
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@@
+    (effects (font (size 1.5 1.5) (thickness 0.3)) (justify left mirror))
+  )
+  (gr_text "Battery" (at 149 81) (layer "B.SilkS")
     (effects (font (size 1.5 1.5) (thickness 0.3)) (justify left mirror))
   )
