File: pcb/moisture-sensor.kicad_sch (KiCad schematic)
At the start: 35 parts, among them J3 USB4110, U1 ESP32-C3-WROOM-02, U2 TPS631000, U4 MCP73832, Y1 32.768kHz

Commit message: improve PCB
Parts:
- RESET1: footprint library:Panasonic_Electronic_Components-EVQ-P2202M-MFG -> Button_Switch_SMD:SW_SPST_EVQP2; symbol EVQ-P2202M:EVQ-P2202M -> Switch:SW_Push
- U2: footprint friedrich:SOT-583 -> Package_TO_SOT_SMD:SC-70-8
Connections:
- net GND: now also RESET1.1; no longer RESET1.2
- net at R4.1: now also RESET1.2; no longer RESET1.1
Changed lines of the file:
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@@
     (stroke (width 0) (type default) (color 0 0 0 0))
   )
-  (wire (pts (xy 73.66 124.46) (xy 73.66 138.43))
+  (wire (pts (xy 78.74 124.46) (xy 78.74 138.43))
     (stroke (width 0) (type default) (color 0 0 0 0))
   )
@@
     (stroke (width 0) (type default) (color 0 0 0 0))
   )
-  (wire (pts (xy 73.66 124.46) (xy 81.28 124.46))
+  (wire (pts (xy 78.74 124.46) (xy 81.28 124.46))
     (stroke (width 0) (type default) (color 0 0 0 0))
   )
@@
     (pin "2")
   )
-  (symbol (lib_id "EVQ-P2202M:EVQ-P2202M") (at 81.28 121.92 0) (unit 1)
+  (symbol (lib_id "Switch:SW_Push") (at 86.36 124.46 0) (unit 1)
     (in_bom yes) (on_board yes)
-    (property "Reference" "RESET1" (id 0) (at 86.36 121.92 0))
-    (property "Value" "EVQ-Q2F03W" (id 1) (at 85.09 121.92 0)
-      (effects (font (size 1.27 1.27)) hide)
-    )
-    (property "Footprint" "library:Panasonic_Electronic_Components-EVQ-P2202M-MFG" (id 2) (at 81.28 116.84 0)
-      (effects (font (size 1.27 1.27)) (justify left) hide)
-    )
-    (property "Datasheet" "https://industrial.panasonic.com/ac/cdn/e/control/switch/light-touch/catalog/sw_lt_eng_4735s.pdf" (id 3) (at 81.28 114.3 0)
-      (effects (font (size 1.27 1.27)) (justify left) hide)
-    )
-    (property "MPN" "EVQ-Q2F03W" (id 4) (at 81.28 121.92 0)
-      (effects (font (size 1.27 1.27)) hide)
-    )
-    (pin "1")
-    (pin "2")
-    (pin "3")
-    (pin "4")
+    (property "Reference" "RESET1" (id 0) (at 86.36 119.38 0))
+    (property "Value" "EVQ-Q2F03W" (id 1) (at 90.17 124.46 0)
+      (effects (font (size 1.27 1.27)) hide)
+    )
+    (property "Footprint" "Button_Switch_SMD:SW_SPST_EVQP2" (id 2) (at 86.36 119.38 0)
+      (effects (font (size 1.27 1.27)) hide)
+    )
+    (property "Datasheet" "~" (id 3) (at 86.36 119.38 0)
+      (effects (font (size 1.27 1.27)) hide)
+    )
+    (property "MPN" "EVQ-Q2F03W" (id 4) (at 86.36 124.46 0)
+      (effects (font (size 1.27 1.27)) hide)
+    )
+    (pin "1")
+    (pin "2")
   )
   (symbol (lib_id "power:GND") (at 52.07 91.44 0) (unit 1)
@@
     (pin "2")
   )
-  (symbol (lib_id "power:GND") (at 73.66 138.43 0) (unit 1)
-    (in_bom yes) (on_board yes) (fields_autoplaced)
-    (property "Reference" "#PWR0104" (id 0) (at 73.66 144.78 0)
-      (effects (font (size 1.27 1.27)) hide)
-    )
-    (property "Value" "GND" (id 1) (at 73.66 143.51 0))
-    (property "Footprint" "" (id 2) (at 73.66 138.43 0)
-      (effects (font (size 1.27 1.27)) hide)
-    )
-    (property "Datasheet" "" (id 3) (at 73.66 138.43 0)
+  (symbol (lib_id "power:GND") (at 78.74 138.43 0) (unit 1)
+    (in_bom yes) (on_board yes) (fields_autoplaced)
+    (property "Reference" "#PWR0104" (id 0) (at 78.74 144.78 0)
+      (effects (font (size 1.27 1.27)) hide)
+    )
+    (property "Value" "GND" (id 1) (at 78.74 143.51 0))
+    (property "Footprint" "" (id 2) (at 78.74 138.43 0)
+      (effects (font (size 1.27 1.27)) hide)
+    )
+    (property "Datasheet" "" (id 3) (at 78.74 138.43 0)
       (effects (font (size 1.27 1.27)) hide)
     )
@@
     (property "Reference" "U2" (id 0) (at 209.55 121.92 0))
     (property "Value" "TPS631000" (id 1) (at 209.55 124.46 0))
-    (property "Footprint" "friedrich:SOT-583" (id 2) (at 207.01 123.19 0)
+    (property "Footprint" "Package_TO_SOT_SMD:SC-70-8" (id 2) (at 207.01 123.19 0)
       (effects (font (size 1.27 1.27)) hide)
     )
@@
     )
     (path "/4d1b128f-a7a4-4f89-9e1f-a12bb17f1956"
-      (reference "RESET1") (unit 1) (value "EVQ-Q2F03W") (footprint "library:Panasonic_Electronic_Components-EVQ-P2202M-MFG")
+      (reference "RESET1") (unit 1) (value "EVQ-Q2F03W") (footprint "Button_Switch_SMD:SW_SPST_EVQP2")
     )
     (path "/fa898b87-1714-4bd5-8bc1-596ed62b5578"
@@
     )
     (path "/87d0a414-90d1-4b10-a9e6-0eae005dda6c"
-      (reference "U2") (unit 1) (value "TPS631000") (footprint "friedrich:SOT-583")
+      (reference "U2") (unit 1) (value "TPS631000") (footprint "Package_TO_SOT_SMD:SC-70-8")
     )
     (path "/fd1a9b7d-95bf-4223-b0f2-0725a8ad4579"

Commit message: add footprints and 3d models, increase solder pad size
Parts:
- J3: footprint GCT_USB4110-GF-A_REVB -> library:GCT_USB4110-GF-A_REVB
- U1: footprint Espressif:ESP32-C3-WROOM-02 -> library:ESP32-C3-WROOM-02
- Y1: footprint XTAL_ABS07-32.768KHZ-1-T -> library:ABS07-32.768KHZ-T
Other:
- note added: "Crystal"
- note removed: "Oscillator"
Changed lines of the file:
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@@
     (effects (font (size 2.5 2.5)) (justify left bottom))
   )
-  (text "Oscillator" (at 22.86 105.41 0)
+  (text "Crystal" (at 22.86 105.41 0)
     (effects (font (size 2.5 2.5)) (justify left bottom))
   )
@@
     (property "Reference" "Y1" (id 0) (at 31.75 116.84 0))
     (property "Value" "32.768kHz" (id 1) (at 31.75 119.38 0))
-    (property "Footprint" "XTAL_ABS07-32.768KHZ-1-T" (id 2) (at 31.75 124.46 0)
+    (property "Footprint" "library:ABS07-32.768KHZ-T" (id 2) (at 31.75 124.46 0)
       (effects (font (size 1.27 1.27)) (justify left bottom) hide)
     )
@@
     (property "Reference" "J3" (id 0) (at 118.11 154.94 0))
     (property "Value" "USB4110" (id 1) (at 118.11 157.48 0))
-    (property "Footprint" "GCT_USB4110-GF-A_REVB" (id 2) (at 118.11 170.18 0)
+    (property "Footprint" "library:GCT_USB4110-GF-A_REVB" (id 2) (at 118.11 170.18 0)
       (effects (font (size 1.27 1.27)) (justify left bottom) hide)
     )
@@
     (property "Reference" "U1" (id 0) (at 100.965 22.86 0))
     (property "Value" "ESP32-C3-WROOM-02" (id 1) (at 100.965 25.4 0))
-    (property "Footprint" "Espressif:ESP32-C3-WROOM-02" (id 2) (at 100.33 92.71 0)
+    (property "Footprint" "library:ESP32-C3-WROOM-02" (id 2) (at 100.33 92.71 0)
       (effects (font (size 1.27 1.27)) hide)
     )
@@
     )
     (path "/e1852524-e042-4a79-89b8-c137524f4cbd"
-      (reference "J3") (unit 1) (value "USB4110") (footprint "GCT_USB4110-GF-A_REVB")
+      (reference "J3") (unit 1) (value "USB4110") (footprint "library:GCT_USB4110-GF-A_REVB")
     )
     (path "/6854da47-4f08-4419-af98-9e6336d90815"
@@
     )
     (path "/fa898b87-1714-4bd5-8bc1-596ed62b5578"
-      (reference "U1") (unit 1) (value "ESP32-C3-WROOM-02") (footprint "Espressif:ESP32-C3-WROOM-02")
+      (reference "U1") (unit 1) (value "ESP32-C3-WROOM-02") (footprint "library:ESP32-C3-WROOM-02")
     )
     (path "/87d0a414-90d1-4b10-a9e6-0eae005dda6c"
@@
     )
     (path "/98cb8a72-5f9e-47a5-9051-d93a01408421"
-      (reference "Y1") (unit 1) (value "32.768kHz") (footprint "XTAL_ABS07-32.768KHZ-1-T")
-    )
-  )
+      (reference "Y1") (unit 1) (value "32.768kHz") (footprint "library:ABS07-32.768KHZ-T")
+    )
+  )

Commit message: adjust some component values
Parts:
- C4: value 22uF -> 47uF; MPN GRM21BZ71A226ME15 -> GRM21BR61A476ME15
- R12: value 120R -> 220R; MPN RC0805FR-07120RL -> RC0805FR-07220RL
Changed lines of the file:
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@@
       (effects (font (size 1.27 1.27)) (justify right))
     )
-    (property "Value" "120R" (id 1) (at 177.8 54.6099 0)
+    (property "Value" "220R" (id 1) (at 177.8 54.6099 0)
       (effects (font (size 1.27 1.27)) (justify right))
     )
@@
       (effects (font (size 1.27 1.27)) hide)
     )
-    (property "MPN" "RC0805FR-07120RL" (id 4) (at 175.26 53.34 0)
+    (property "MPN" "RC0805FR-07220RL" (id 4) (at 175.26 53.34 0)
       (effects (font (size 1.27 1.27)) hide)
     )
@@
       (effects (font (size 1.27 1.27)) (justify left))
     )
-    (property "Value" "22uF" (id 1) (at 191.77 144.7799 0)
+    (property "Value" "47uF" (id 1) (at 191.77 144.7799 0)
       (effects (font (size 1.27 1.27)) (justify left))
     )
@@
       (effects (font (size 1.27 1.27)) hide)
     )
-    (property "MPN" "GRM21BZ71A226ME15" (id 4) (at 187.96 143.51 0)
+    (property "MPN" "GRM21BR61A476ME15" (id 4) (at 187.96 143.51 0)
       (effects (font (size 1.27 1.27)) hide)
     )
@@
     )
     (path "/ba9a2a55-7b19-46a7-86ca-7630aa58a059"
-      (reference "C4") (unit 1) (value "22uF") (footprint "Capacitor_SMD:C_0805_2012Metric_Pad1.18x1.45mm_HandSolder")
+      (reference "C4") (unit 1) (value "47uF") (footprint "Capacitor_SMD:C_0805_2012Metric_Pad1.18x1.45mm_HandSolder")
     )
     (path "/e14e10b8-5142-473e-a2c0-7284a4b8625c"
@@
     )
     (path "/3ae33bbc-cc68-4c60-94fc-bc559776b4f5"
-      (reference "R12") (unit 1) (value "120R") (footprint "Resistor_SMD:R_0805_2012Metric_Pad1.20x1.40mm_HandSolder")
+      (reference "R12") (unit 1) (value "220R") (footprint "Resistor_SMD:R_0805_2012Metric_Pad1.20x1.40mm_HandSolder")
     )
     (path "/59f24728-e1d5-49ea-a06b-e5d3361459fe"

Commit message: fix reset button
Parts:
- RESET1: MPN EVQ-Q2F03W -> EVQ-P2K02Q
Changed lines of the file:
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@@
       (effects (font (size 1.27 1.27)) hide)
     )
-    (property "MPN" "EVQ-Q2F03W" (id 4) (at 86.36 124.46 0)
+    (property "MPN" "EVQ-P2K02Q" (id 4) (at 86.36 124.46 0)
       (effects (font (size 1.27 1.27)) hide)
     )
